Commit message: adding RGB-D camera

File: chaser_robot/urdf/chaser_robot.xacro (robot description, xacro)
@@ -119,5 +119,5 @@
     <dynamics damping="1.0" friction="1.0"/>
   </joint>
-  <link name="camera">
+  <link name="camera_link">
       <inertial>
         <origin xyz="0.0 0.0 0.0" rpy="0.0 0.0 0.0"/>
@@ -137,5 +137,5 @@
         </geometry>
       </collision>
-      <gazebo reference="camera">
+      <gazebo reference="camera_link">
           <material>Gazebo/Green</material>
       </gazebo>
@@ -144,7 +144,14 @@
     <origin xyz="0.2 0.0 0.0" rpy="0.0 0.0 0.0"/>
     <parent link="chassis"/>
-    <child link="camera"/>
+    <child link="camera_link"/>
     <axis xyz="0.0 1 0.0"/>
   </joint>
+  <joint name="camera_optical_joint" type="fixed">
+    <origin xyz="0 0 0" rpy="-1.5707 0 -1.5707"/>
+    <parent link="camera_link"/>
+    <child link="camera_link_optical"/>
+  </joint>
+  <link name="camera_link_optical">
+  </link>
   <link name="hokuyo">
       <inertial>
